Commit message: namespace setting

File: minibot_description/urdf/file/1/minibot.urdf.xacro (robot description, xacro)
@@ -3,11 +3,11 @@
     <xacro:macro name="insert_robot" params="prefix">
         <xacro:property name="wheel_diameter" value="0.068"/>
-        <xacro:property name="wheel_seperation" value="0.180"/>
-        <link name="base_footprint"/>
-        <link name="base_link">
+        <xacro:property name="wheel_speration" value="0.180"/>
+        <link name="${prefix}base_footprint"/>
+        <link name="${prefix}base_link">
             <visual>
                 <origin xyz="0 0 0" rpy="0 0 0"/>
                 <geometry>
-                    <mesh filename="file://$(find minibot_description)/meshes/visual/base_link.dae" scale="1 1 1"/>
+                    <mesh filename="file://$(find rmf_pinklab_assets)/meshes/minibot/visual/base_link.dae" scale="1 1 1"/>
                 </geometry>
             </visual>
@@ -15,5 +15,5 @@
                 <origin xyz="0 0 0" rpy="0 0 0"/>
                 <geometry>
-                    <mesh filename="file://$(find minibot_description)/meshes/collision/base_link.stl" scale="1 1 1"/>
+                    <mesh filename="file://$(find rmf_pinklab_assets)/meshes/minibot/collision/base_link.stl" scale="1 1 1"/>
                 </geometry>
             </collision>
@@ -25,15 +25,15 @@
             </inertial>
         </link>
-        <joint name="base_link_fixed_joint" type="fixed">
-            <parent link="base_footprint"/>
-            <child link="base_link"/>
+        <joint name="${prefix}base_link_fixed_joint" type="fixed">
+            <parent link="${prefix}base_footprint"/>
+            <child link="${prefix}base_link"/>
             <origin xyz="0 0 ${wheel_diameter/2}" rpy="0 0 0"/>
         </joint>
         <xacro:macro name="insert_wheel" params="parent prefix prefix_dir dir">
-            <link name="${prefix_dir}_wheel">
+            <link name="${prefix}${prefix_dir}_wheel">
                 <visual>
                     <origin xyz="0 0 0" rpy="0 0 ${dir * pi/2}"/>
                     <geometry>
-                        <mesh filename="file://$(find minibot_description)/meshes/visual/wheel.dae" scale="1 1 1"/>
+                        <mesh filename="file://$(find rmf_pinklab_assets)/meshes/minibot/visual/wheel.dae" scale="1 1 1"/>
                     </geometry>
                 </visual>
@@ -41,5 +41,5 @@
                     <origin xyz="0 0 0" rpy="0 0 ${dir * pi/2}"/>
                     <geometry>
-                        <mesh filename="file://$(find minibot_description)/meshes/collision/wheel.stl" scale="1 1 1"/>
+                        <mesh filename="file://$(find rmf_pinklab_assets)/meshes/minibot/collision/wheel.stl" scale="1 1 1"/>
                     </geometry>
                 </collision>
@@ -52,18 +52,18 @@
                 </inertial>
             </link>
-            <joint name="${prefix_dir}_wheel_joint" type="continuous">
+            <joint name="${prefix}${prefix_dir}_wheel_joint" type="continuous">
                 <parent link="${parent}"/>
-                <child link="${prefix_dir}_wheel"/>
+                <child link="${prefix}${prefix_dir}_wheel"/>
                 <axis xyz="0 1 0"/>
-                <origin xyz="0 ${dir * wheel_seperation/2} 0" rpy="0 0 0"/>
+                <origin xyz="0 ${dir * wheel_speration/2} 0" rpy="0 0 0"/>
             </joint>
         </xacro:macro>
-        <xacro:insert_wheel parent="base_link" prefix="" prefix_dir="l" dir="1" />
-        <xacro:insert_wheel parent="base_link" prefix="" prefix_dir="r" dir="-1" />
-        <link name="front_camera_mount">
+        <xacro:insert_wheel parent="${prefix}base_link" prefix="${prefix}" prefix_dir="l" dir="1" />
+        <xacro:insert_wheel parent="${prefix}base_link" prefix="${prefix}" prefix_dir="r" dir="-1" />
+        <link name="${prefix}front_camera_mount">
             <visual>
                 <origin xyz="0 0 0" rpy="0 0 0"/>
                 <geometry>
-                    <mesh filename="file://$(find minibot_description)/meshes/visual/front_camera.dae" scale="1 1 1"/>
+                    <mesh filename="file://$(find rmf_pinklab_assets)/meshes/minibot/visual/front_camera.dae" scale="1 1 1"/>
                 </geometry>
             </visual>
@@ -71,5 +71,5 @@
                 <origin xyz="0 0 0" rpy="0 0 0"/>
                 <geometry>
-                    <mesh filename="file://$(find minibot_description)/meshes/collision/front_camera.stl" scale="1 1 1"/>
+                    <mesh filename="file://$(find rmf_pinklab_assets)/meshes/minibot/collision/front_camera.stl" scale="1 1 1"/>
                 </geometry>
             </collision>
@@ -80,20 +80,20 @@
             </inertial>
         </link>
-        <joint name="front_camera_mount_fixed_joint" type="fixed">
-            <parent link="base_link"/>
-            <child link="front_camera_mount"/>
+        <joint name="${prefix}front_camera_mount_fixed_joint" type="fixed">
+            <parent link="${prefix}base_link"/>
+            <child link="${prefix}front_camera_mount"/>
             <origin xyz="0.045 0 0.085" rpy="0 0 0"/>
         </joint>
-        <link name="camera_link"/>
-        <joint name="camera_link_fixed_joint" type="fixed">
-            <parent link="front_camera_mount"/>
-            <child link="camera_link"/>
+        <link name="${prefix}camera_link"/>
+        <joint name="${prefix}camera_link_fixed_joint" type="fixed">
+            <parent link="${prefix}front_camera_mount"/>
+            <child link="${prefix}camera_link"/>
             <origin xyz="0.0111 0 0.0193" rpy="0 ${pi/2} 0"/>
         </joint>
-        <link name="ul_sensor_mount">
+        <link name="${prefix}ul_sensor_mount">
             <visual>
                 <origin xyz="0 0 0" rpy="0 0 0"/>
                 <geometry>
-                    <mesh filename="file://$(find minibot_description)/meshes/visual/ul_sensor.dae" scale="1 1 1"/>
+                    <mesh filename="file://$(find rmf_pinklab_assets)/meshes/minibot/visual/ul_sensor.dae" scale="1 1 1"/>
                 </geometry>
             </visual>
@@ -101,5 +101,5 @@
                 <origin xyz="0 0 0" rpy="0 0 0"/>
                 <geometry>
-                    <mesh filename="file://$(find minibot_description)/meshes/collision/ul_sensor.stl" scale="1 1 1"/>
+                    <mesh filename="file://$(find rmf_pinklab_assets)/meshes/minibot/collision/ul_sensor.stl" scale="1 1 1"/>
                 </geometry>
             </collision>
@@ -110,13 +110,13 @@
             </inertial>
         </link>
-        <joint name="ul_sensor_mount_fixed_joint" type="fixed">
-            <parent link="base_link"/>
-            <child link="ul_sensor_mount"/>
+        <joint name="${prefix}ul_sensor_mount_fixed_joint" type="fixed">
+            <parent link="${prefix}base_link"/>
+            <child link="${prefix}ul_sensor_mount"/>
             <origin xyz="0.03 0 0.01" rpy="0 0 0"/>
         </joint>
-        <link name="ul_sensor_link"/>
-        <joint name="ul_sensor_link_fixed_joint" type="fixed">
-            <parent link="ul_sensor_mount"/>
-            <child link="ul_sensor_link"/>
+        <link name="${prefix}ul_sensor_link"/>
+        <joint name="${prefix}ul_sensor_link_fixed_joint" type="fixed">
+            <parent link="${prefix}ul_sensor_mount"/>
+            <child link="${prefix}ul_sensor_link"/>
             <origin xyz="0.02 0 0" rpy="0 0 0"/>
         </joint>

File: minibot_description/urdf/file/1/minibot_gazebo.urdf.xacro (robot description, xacro)
@@ -4,14 +4,8 @@
         <gazebo>
             <plugin filename="libgazebo_ros2_control.so" name="gazebo_ros2_control">
-                <ros>
-                    <namespace>/${prefix}</namespace>
-                    <remapping>/tf:=tf</remapping>
-                    <remapping>/tf_static:=tf_static</remapping>
-                    <!-- <remapping>/odom:=/base_controller/odom</remapping> -->
-                  </ros>
-                <parameters>$(find minibot_bringup)/config/minibot_controllers_gazebo.yaml</parameters>
+                <parameters>$(find rmf_pinklab_assets)/config/minibot_controllers_gazebo.yaml</parameters>
             </plugin>
         </gazebo>
-        <gazebo reference="l_wheel">
+        <gazebo reference="${prefix}l_wheel">
             <mu1>200</mu1>
             <mu2>200</mu2>
@@ -20,5 +14,5 @@
             <!-- <minDepth>0.001</minDepth> -->
         </gazebo>
-        <gazebo reference="r_wheel">
+        <gazebo reference="${prefix}r_wheel">
             <mu1>200</mu1>
             <mu2>200</mu2>
@@ -27,10 +21,10 @@
             <!-- <minDepth>0.001</minDepth> -->
         </gazebo>
-        <gazebo reference="base_link">
+        <gazebo reference="${prefix}base_link">
             <mu1>0.0</mu1>
             <mu2>0.0</mu2>
             <!-- <minDepth>0.001</minDepth> -->
         </gazebo>
-        <gazebo reference="laser_link">
+        <gazebo reference="${prefix}laser_link">
             <sensor name="laser" type="ray">
                 <pose>0 0 0 0 0 0</pose>
@@ -60,16 +54,15 @@
                 <plugin name="laser" filename="libgazebo_ros_ray_sensor.so">
                     <ros>
-                        <namespace>${prefix}</namespace>
                         <remapping>~/out:=scan</remapping>
                     </ros>
-                    <frame_name>laser_link</frame_name>
+                    <frame_name>${prefix}laser_link</frame_name>
                     <output_type>sensor_msgs/LaserScan</output_type>
                 </plugin>
             </sensor>
         </gazebo>
-        <!-- <gazebo reference="camera_link">
-            <sensor name="camera" type="camera">
+        <gazebo reference="${prefix}camera_link">
+            <sensor name="${prefix}camera" type="camera">
                 <update_rate>30.0</update_rate>
-                <camera name="camera">
+                <camera name="${prefix}camera">
                     <pose>0 0 0 0 -1.5707 0</pose>
                     <horizontal_fov>1.08</horizontal_fov>
@@ -89,9 +82,9 @@
                     </noise>
                 </camera>
-                <plugin name="camera_controller" filename="libgazebo_ros_camera.so">
+                <plugin name="${prefix}camera_controller" filename="libgazebo_ros_camera.so">
                     <ros>
-                        <namespace>camera</namespace>
-                        <remapping>camera1/image_raw:=camera/image_test</remapping>
-                        <remapping>camera_info:=camera_info_test</remapping>
+                        <!-- <namespace>${prefix}camera</namespace> -->
+                        <!-- <remapping>camera1/image_raw:=camera/image_test</remapping>
+                        <remapping>camera_info:=camera_info_test</remapping> -->
                     </ros>
                     <frame_name>camera_link</frame_name>
@@ -99,5 +92,5 @@
                 </plugin>
             </sensor>
-        </gazebo> -->
+        </gazebo>
     </xacro:macro>
 </robot>

File: minibot_description/urdf/file/1/minibot_ros2_control.urdf.xacro (robot description, xacro)
@@ -1,6 +1,6 @@
 <?xml version="1.0"?>
 <robot xmlns:xacro="http://www.ros.org/wiki/xacro">
-    <xacro:macro name="insert_ros2_control" params="prefix is_sim:=false robot_port_name robot_baudrate">
-        <ros2_control name="${prefix}/minibot_system" type="system">
+    <xacro:macro name="insert_ros2_control" params="prefix is_sim:=^|false robot_port_name robot_baudrate">
+        <ros2_control name="${prefix}minibot_system" type="system">
             <xacro:if value="$(arg is_sim)">
                 <hardware>
@@ -15,5 +15,5 @@
                 </hardware>
             </xacro:unless>
-            <joint name="l_wheel_joint">
+            <joint name="${prefix}l_wheel_joint">
                 <command_interface name="velocity">
                     <param name="min">-1.0</param>
@@ -23,5 +23,5 @@
                 <state_interface name="velocity"/>
             </joint>
-            <joint name="r_wheel_joint">
+            <joint name="${prefix}r_wheel_joint">
                 <command_interface name="velocity">
                     <param name="min">-1.0</param>

File: minibot_description/urdf/file/1/robot.urdf.xacro (robot description, xacro)
@@ -1,8 +1,8 @@
 <?xml version="1.0"?>
-<robot xmlns:xacro="http://ros.org/wiki/xacro" name="minibot">
-    <xacro:include filename="$(find minibot_description)/urdf/common/inertia_macro.urdf.xacro"/>
-    <xacro:include filename="$(find minibot_description)/urdf/minibot.urdf.xacro"/>
-    <xacro:include filename="$(find minibot_description)/urdf/minibot_gazebo.urdf.xacro"/>
-    <xacro:include filename="$(find minibot_description)/urdf/minibot_ros2_control.urdf.xacro"/>
+<robot xmlns:xacro="http://ros.org/wiki/xacro" name="aidl200">
+    <xacro:include filename="$(find rmf_pinklab_assets)/urdf/common/inertia_macro.urdf.xacro"/>
+    <xacro:include filename="$(find rmf_pinklab_assets)/urdf/minibot/minibot.urdf.xacro"/>
+    <xacro:include filename="$(find rmf_pinklab_assets)/urdf/minibot/minibot_gazebo.urdf.xacro"/>
+    <xacro:include filename="$(find rmf_pinklab_assets)/urdf/minibot/minibot_ros2_control.urdf.xacro"/>
     <xacro:arg name="prefix" default=""/>
     <xacro:arg name="is_sim" default="false"/>
@@ -17,9 +17,9 @@
     </xacro:if>
     <!-- insert ydlidar_x2 lidar -->
-    <link name="ydlidar_lidar_mount">
+    <link name="${prefix}ydlidar_lidar_mount">
         <visual>
             <origin xyz="0 0 0" rpy="0 0 0"/>
             <geometry>
-                <mesh filename="file://$(find minibot_description)/meshes/visual/ydlidar_x2_assy.dae" scale="1 1 1"/>
+                <mesh filename="file://$(find rmf_pinklab_assets)/meshes/minibot/visual/ydlidar_x2_assy.dae" scale="1 1 1"/>
             </geometry>
         </visual>
@@ -27,5 +27,5 @@
             <origin xyz="0 0 0" rpy="0 0 0"/>
             <geometry>
-                <mesh filename="file://$(find minibot_description)/meshes/collision/ydlidar_x2_assy.stl" scale="1 1 1"/>
+                <mesh filename="file://$(find rmf_pinklab_assets)/meshes/minibot/collision/ydlidar_x2_assy.stl" scale="1 1 1"/>
             </geometry>
         </collision>
@@ -36,13 +36,13 @@
         </inertial>
     </link>
-    <joint name="ydidar_mount_fixed_joint" type="fixed">
-        <parent link="base_link"/>
-        <child link="ydlidar_lidar_mount"/>
+    <joint name="${prefix}idar_mount_fixed_joint" type="fixed">
+        <parent link="${prefix}base_link"/>
+        <child link="${prefix}ydlidar_lidar_mount"/>
         <origin xyz="-0.01 0 0.085" rpy="0 0 0"/>
     </joint>
-    <link name="laser_link"/>
-    <joint name="laser_link_fixed_joint" type="fixed">
-        <parent link="ydlidar_lidar_mount"/>
-        <child link="laser_link"/>
+    <link name="${prefix}laser_link"/>
+    <joint name="${prefix}laser_link_fixed_joint" type="fixed">
+        <parent link="${prefix}ydlidar_lidar_mount"/>
+        <child link="${prefix}laser_link"/>
         <origin xyz="0 0 0.04245" rpy="0 0 0"/>
     </joint>

File: minibot_description/urdf/file/minibot_gazebo.urdf.xacro (robot description, xacro)
@@ -4,14 +4,8 @@
         <gazebo>
             <plugin filename="libgazebo_ros2_control.so" name="gazebo_ros2_control">
-                <ros>
-                    <namespace>/${prefix}</namespace>
-                    <remapping>/tf:=tf</remapping>
-                    <remapping>/tf_static:=tf_static</remapping>
-                    <!-- <remapping>/odom:=/base_controller/odom</remapping> -->
-                  </ros>
-                <parameters>$(find minibot_bringup)/config/minibot_controllers_gazebo.yaml</parameters>
+                <parameters>$(find rmf_pinklab_assets)/config/minibot_controllers_gazebo.yaml</parameters>
             </plugin>
         </gazebo>
-        <gazebo reference="l_wheel">
+        <gazebo reference="${prefix}/l_wheel">
             <mu1>200</mu1>
             <mu2>200</mu2>
@@ -20,5 +14,5 @@
             <!-- <minDepth>0.001</minDepth> -->
         </gazebo>
-        <gazebo reference="r_wheel">
+        <gazebo reference="${prefix}/r_wheel">
             <mu1>200</mu1>
             <mu2>200</mu2>
@@ -27,10 +21,10 @@
             <!-- <minDepth>0.001</minDepth> -->
         </gazebo>
-        <gazebo reference="base_link">
+        <gazebo reference="${prefix}/base_link">
             <mu1>0.0</mu1>
             <mu2>0.0</mu2>
             <!-- <minDepth>0.001</minDepth> -->
         </gazebo>
-        <gazebo reference="laser_link">
+        <gazebo reference="${prefix}/laser_link">
             <sensor name="laser" type="ray">
                 <pose>0 0 0 0 0 0</pose>
@@ -60,16 +54,15 @@
                 <plugin name="laser" filename="libgazebo_ros_ray_sensor.so">
                     <ros>
-                        <namespace>${prefix}</namespace>
                         <remapping>~/out:=scan</remapping>
                     </ros>
-                    <frame_name>laser_link</frame_name>
+                    <frame_name>${prefix}/laser_link</frame_name>
                     <output_type>sensor_msgs/LaserScan</output_type>
                 </plugin>
             </sensor>
         </gazebo>
-        <!-- <gazebo reference="camera_link">
-            <sensor name="camera" type="camera">
+        <gazebo reference="${prefix}/camera_link">
+            <sensor name="${prefix}/camera" type="camera">
                 <update_rate>30.0</update_rate>
-                <camera name="camera">
+                <camera name="${prefix}/camera">
                     <pose>0 0 0 0 -1.5707 0</pose>
                     <horizontal_fov>1.08</horizontal_fov>
@@ -89,9 +82,9 @@
                     </noise>
                 </camera>
-                <plugin name="camera_controller" filename="libgazebo_ros_camera.so">
+                <plugin name="${prefix}/camera_controller" filename="libgazebo_ros_camera.so">
                     <ros>
-                        <namespace>camera</namespace>
-                        <remapping>camera1/image_raw:=camera/image_test</remapping>
-                        <remapping>camera_info:=camera_info_test</remapping>
+                        <!-- <namespace>${prefix}/camera</namespace> -->
+                        <!-- <remapping>camera1/image_raw:=camera/image_test</remapping>
+                        <remapping>camera_info:=camera_info_test</remapping> -->
                     </ros>
                     <frame_name>camera_link</frame_name>
@@ -99,5 +92,5 @@
                 </plugin>
             </sensor>
-        </gazebo> -->
+        </gazebo>
     </xacro:macro>
 </robot>

File: minibot_description/urdf/file/minibot_ros2_control.urdf.xacro (robot description, xacro)
@@ -15,5 +15,5 @@
                 </hardware>
             </xacro:unless>
-            <joint name="l_wheel_joint">
+            <joint name="${prefix}/l_wheel_joint">
                 <command_interface name="velocity">
                     <param name="min">-1.0</param>
@@ -23,5 +23,5 @@
                 <state_interface name="velocity"/>
             </joint>
-            <joint name="r_wheel_joint">
+            <joint name="${prefix}/r_wheel_joint">
                 <command_interface name="velocity">
                     <param name="min">-1.0</param>

File: minibot_description/urdf/file/robot.urdf.xacro (robot description, xacro)
@@ -1,8 +1,8 @@
 <?xml version="1.0"?>
-<robot xmlns:xacro="http://ros.org/wiki/xacro" name="minibot">
-    <xacro:include filename="$(find minibot_description)/urdf/common/inertia_macro.urdf.xacro"/>
-    <xacro:include filename="$(find minibot_description)/urdf/minibot.urdf.xacro"/>
-    <xacro:include filename="$(find minibot_description)/urdf/minibot_gazebo.urdf.xacro"/>
-    <xacro:include filename="$(find minibot_description)/urdf/minibot_ros2_control.urdf.xacro"/>
+<robot xmlns:xacro="http://ros.org/wiki/xacro" name="aidl200">
+    <xacro:include filename="$(find rmf_pinklab_assets)/urdf/common/inertia_macro.urdf.xacro"/>
+    <xacro:include filename="$(find rmf_pinklab_assets)/urdf/minibot/minibot.urdf.xacro"/>
+    <xacro:include filename="$(find rmf_pinklab_assets)/urdf/minibot/minibot_gazebo.urdf.xacro"/>
+    <xacro:include filename="$(find rmf_pinklab_assets)/urdf/minibot/minibot_ros2_control.urdf.xacro"/>
     <xacro:arg name="prefix" default=""/>
     <xacro:arg name="is_sim" default="false"/>
@@ -17,9 +17,9 @@
     </xacro:if>
     <!-- insert ydlidar_x2 lidar -->
-    <link name="ydlidar_lidar_mount">
+    <link name="${prefix}/ydlidar_lidar_mount">
         <visual>
             <origin xyz="0 0 0" rpy="0 0 0"/>
             <geometry>
-                <mesh filename="file://$(find minibot_description)/meshes/visual/ydlidar_x2_assy.dae" scale="1 1 1"/>
+                <mesh filename="file://$(find rmf_pinklab_assets)/meshes/minibot/visual/ydlidar_x2_assy.dae" scale="1 1 1"/>
             </geometry>
         </visual>
@@ -27,5 +27,5 @@
             <origin xyz="0 0 0" rpy="0 0 0"/>
             <geometry>
-                <mesh filename="file://$(find minibot_description)/meshes/collision/ydlidar_x2_assy.stl" scale="1 1 1"/>
+                <mesh filename="file://$(find rmf_pinklab_assets)/meshes/minibot/collision/ydlidar_x2_assy.stl" scale="1 1 1"/>
             </geometry>
         </collision>
@@ -36,13 +36,13 @@
         </inertial>
     </link>
-    <joint name="ydidar_mount_fixed_joint" type="fixed">
-        <parent link="base_link"/>
-        <child link="ydlidar_lidar_mount"/>
+    <joint name="${prefix}/idar_mount_fixed_joint" type="fixed">
+        <parent link="${prefix}/base_link"/>
+        <child link="${prefix}/ydlidar_lidar_mount"/>
         <origin xyz="-0.01 0 0.085" rpy="0 0 0"/>
     </joint>
-    <link name="laser_link"/>
-    <joint name="laser_link_fixed_joint" type="fixed">
-        <parent link="ydlidar_lidar_mount"/>
-        <child link="laser_link"/>
+    <link name="${prefix}/laser_link"/>
+    <joint name="${prefix}/laser_link_fixed_joint" type="fixed">
+        <parent link="${prefix}/ydlidar_lidar_mount"/>
+        <child link="${prefix}/laser_link"/>
         <origin xyz="0 0 0.04245" rpy="0 0 0"/>
     </joint>
